File: ABU2025-IBT_2.kicad_sch (KiCad schematic)
At the start: 10 parts, among them M1 Motor_DC, Q1 2N4401, Q2 2N4401, U2 ESP32-DevKitM-1

Commit message: Remove unnecessary logic
Parts:
- removed Q1, Q2: 2N4401, Package_TO_SOT_THT:TO-92_Inline, symbol Transistor_Project:2N4401
- removed R1, R2, R3, R4: R, symbol Device:R
Connections:
- net at U1.1 (RPWM): now also U2.31 (GPIO21)
- net at U1.2 (LPWM): now also U2.30 (GPIO22)
